File: SRC/IOT_AGRIFARM_POWER.kicad_sch (KiCad schematic)
At the start: 54 parts, among them Q201 AO3401A, U203 BQ25672RQMR, U206 L78L05, U207 SD8942, U301 DW01A, U303 8205A

Commit message: Version 2 - Added 24V 2A Boost converter for water pump
Parts:
- R213: renamed from R212; value R_Small -> 100K; JLCPCB PART# (none) -> C60491; MANUFACTURER (none) -> YAGEO; MPN (none) -> RC0402FR-07100KL; UNIT PRICE (none) -> 0.0006
- R214: renamed from R213; value R_Small -> 25K5; JLCPCB PART# (none) -> C273695; MANUFACTURER (none) -> YAGEO; MPN (none) -> RC0402FR-0725K5L; UNIT PRICE (none) -> 0.0007
- renumbered R211 to R212
Connections:
- net VSYS renamed +12V
