File: SRC/IoT_Agrifarm.kicad_sch (KiCad schematic)
At the start: 16 parts, among them J101 J_PUMP, J101 USB_C_Receptacle_USB2.0, J102 J_PANEL, J302 Conn_NPK, Q101 AO3401A, Q102 IRLZ44N, U102 AP2171W, U102 USBLC6-2P6

Commit message: Version 2 - Added 24V 2A Boost converter for water pump
Parts:
- removed D101: A7, Diode_SMD:D_SOD-123, symbol Diode:1N4007
- removed Q102: IRLZ44N, Package_TO_SOT_THT:TO-220-3_Vertical, symbol Transistor_FET:IRLZ44N
- removed R205: 100R, Resistor_SMD:R_0603_1608Metric, symbol Device:R
- J101: JLCPCB PART# C2927513 -> C2915641; MPN DB128V-5.08-5P-GN-S -> DB128V-5.08-4P-GN-S; UNIT PRICE 0.3865 -> 0.2883
- J302: footprint Connector_JST:JST_XH_B2B-XH-A_1x02_P2.50mm_Vertical -> Connector_JST:JST_XH_B4B-XH-A_1x04_P2.50mm_Vertical; symbol Connector_Generic:Conn_01x02 -> Connector_Generic:Conn_01x04
- renumbered D102 to D101
Connections:
- net PUMP+ is gone; now on net GND: J101.4 (Pin_4)
- net GND: now also J302.2 (Pin_2); no longer J101.2 (Pin_2)
- net IOT_AGRIFARM_SENSORS/NPK_A: now also J302.3 (Pin_3); no longer J302.1 (Pin_1)
- net IOT_AGRIFARM_SENSORS/NPK_B: now also J302.4 (Pin_4); no longer J302.2 (Pin_2)
- net +24V renamed REGULATOR_SWITCHING_SY7208/VOUT_24V
- net REGULATOR_SWITCHING_SY7208/VOUT_24V: now also J101.2 (Pin_2)
- new net +12V: J302.1 (Pin_1)
Other:
- added sheet REGULATOR_SWITCHING_SY7208 (REGULATOR_SWITCHING_SY7208.kicad_sch)
- note added: "24V BOOST CONVERTER"
